Commit message: Criacao do modelo em URDF
Modelagem da simulação via RVIZ

File: urdf/bres.urdf.xacro (robot description, xacro)
@@ -1,214 +1,85 @@
 <?xml version="1.0"?>
 <robot name="macroed" xmlns:xacro="http://ros.org/wiki/xacro">
-  <xacro:property name="width" value="0.2" />
-  <xacro:property name="leglen" value="0.6" />
-  <xacro:property name="polelen" value="0.2" />
-  <xacro:property name="bodylen" value="0.6" />
-  <xacro:property name="baselen" value="0.4" />
-  <xacro:property name="wheeldiam" value="0.07" />
-  <material name="blue">
+    <xacro:property name="AlturaBase" value="0.0965" />
+    <xacro:property name="AlturaOmbro" value="0.0750" />
+    <xacro:property name="AlturaBraco" value="0.0850" />
+    <xacro:property name="AlturaAntebraco" value="0.0740" />
+    <xacro:property name="AlturaFerramenta" value="0.0300" />
+    <xacro:property name="MedidaPadrao" value="0.1000" />
+    <material name="blue">
     <color rgba="0 0 0.8 1"/>
-  </material>
-  <material name="black">
-    <color rgba="0 0 0 1"/>
-  </material>
-  <material name="white">
-    <color rgba="1 1 1 1"/>
-  </material>
-  <xacro:macro name="default_inertial" params="mass">
-    <inertial>
-      <mass value="${mass}" />
-      <inertia ixx="1e-3" ixy="0.0" ixz="0.0" iyy="1e-3" iyz="0.0" izz="1e-3" />
-    </inertial>
-  </xacro:macro>
-  <link name="base_link">
-    <visual>
-      <geometry>
-        <cylinder radius="${width}" length="${bodylen}"/>
-      </geometry>
-      <material name="blue"/>
-    </visual>
-    <collision>
-      <geometry>
-        <cylinder radius="${width}" length="${bodylen}"/>
-      </geometry>
-    </collision>
-    <xacro:default_inertial mass="10"/>
-  </link>
-  <xacro:macro name="wheel" params="prefix suffix reflect">
-    <link name="${prefix}_${suffix}_wheel">
-      <visual>
-        <origin xyz="0 0 0" rpy="${pi/2} 0 0" />
-        <geometry>
-          <cylinder radius="${wheeldiam/2}" length="0.1"/>
-        </geometry>
-        <material name="black"/>
-      </visual>
-      <collision>
-        <origin xyz="0 0 0" rpy="${pi/2} 0 0" />
-        <geometry>
-          <cylinder radius="${wheeldiam/2}" length="0.1"/>
-        </geometry>
-      </collision>
-      <xacro:default_inertial mass="1"/>
+    </material>
+    <link name="base_link">
+        <visual>
+            <geometry>
+                <cylinder radius="${MedidaPadrao}" length="${AlturaBase}"/>
+            </geometry>
+            <material name="blue"/>
+            <origin xyz="0 0 ${AlturaBase/2}" />
+        </visual>
     </link>
-    <joint name="${prefix}_${suffix}_wheel_joint" type="continuous">
-      <axis xyz="0 1 0" rpy="0 0 0" />
-      <parent link="${prefix}_base"/>
-      <child link="${prefix}_${suffix}_wheel"/>
-      <origin xyz="${baselen*reflect/3} 0 -${wheeldiam/2+.05}" rpy="0 0 0"/>
+    <link name="Ombro">
+        <visual>
+            <geometry>
+                <box size="${MedidaPadrao} ${MedidaPadrao} ${AlturaOmbro}"/>
+            </geometry>
+            <material name="blue"/>
+            <origin xyz="0 0 ${-AlturaOmbro/2}" />
+        </visual>
+    </link>
+    <joint name="base_to_Ombro" type="prismatic">
+        <parent link="base_link"/>
+        <child link="Ombro"/>
+        <limit effort="1000.0" lower="-0.2500" upper="-0.1000" velocity="0.5"/>
+        <axis xyz="0 0 1"/>
+        <origin xyz="0 0 ${AlturaBase}" rpy="${pi} 0 0" />
     </joint>
-  </xacro:macro>
-  <xacro:macro name="leg" params="prefix reflect">
-    <link name="${prefix}_leg">
-      <visual>
-        <geometry>
-          <box size="${leglen} 0.1 0.2"/>
-        </geometry>
-        <origin xyz="0 0 -${leglen/2}" rpy="0 ${pi/2} 0"/>
-        <material name="white"/>
-      </visual>
-      <collision>
-        <geometry>
-          <box size="${leglen} 0.1 0.2"/>
-        </geometry>
-        <origin xyz="0 0 -${leglen/2}" rpy="0 ${pi/2} 0"/>
-      </collision>
-      <xacro:default_inertial mass="10"/>
+    <link name="Braco">
+        <visual>
+            <geometry>
+                <cylinder radius="${MedidaPadrao}" length="${AlturaBraco}"/>
+            </geometry>
+            <material name="blue"/>
+            <origin xyz="0 0 ${-AlturaBraco/2}" />
+        </visual>
     </link>
-    <joint name="base_to_${prefix}_leg" type="fixed">
-      <parent link="base_link"/>
-      <child link="${prefix}_leg"/>
-      <origin xyz="0 ${reflect*(width+.02)} 0.25" />
+    <joint name="Ombro_to_Braco" type="revolute">
+        <parent link="Ombro"/>
+        <child link="Braco"/>
+        <axis xyz="0 0 1"/>
+        <limit effort="1000.0" lower="0.0" upper="0.548" velocity="0.5"/>
+        <origin xyz="0.2500 0 0" />
     </joint>
-    <link name="${prefix}_base">
-      <visual>
-        <geometry>
-          <box size="${baselen} 0.1 0.1"/>
-        </geometry>
-        <material name="white"/>
-      </visual>
-      <collision>
-        <geometry>
-          <box size="${baselen} 0.1 0.1"/>
-        </geometry>
-      </collision>
-      <xacro:default_inertial mass="10"/>
+    <link name="Antebraco">
+        <visual>
+            <geometry>
+                <cylinder radius="${MedidaPadrao}" length="${AlturaAntebraco}"/>
+            </geometry>
+            <material name="blue"/>
+            <origin xyz="0 0 ${-AlturaAntebraco/2}" />
+        </visual>
     </link>
-    <joint name="${prefix}_base_joint" type="fixed">
-      <parent link="${prefix}_leg"/>
-      <child link="${prefix}_base"/>
-      <origin xyz="0 0 ${-leglen}" />
+    <joint name="Braco_to_Antebraco" type="revolute">
+        <parent link="Braco"/>
+        <child link="Antebraco"/>
+        <axis xyz="0 0 1"/>
+        <limit effort="1000.0" lower="0.0" upper="0.548" velocity="0.5"/>
+        <origin xyz="0.2500 0 0" />
     </joint>
-    <xacro:wheel prefix="${prefix}" suffix="front" reflect="1"/>
-    <xacro:wheel prefix="${prefix}" suffix="back" reflect="-1"/>
-  </xacro:macro>
-  <xacro:leg prefix="right" reflect="-1" />
-  <xacro:leg prefix="left" reflect="1" />
-  <joint name="gripper_extension" type="prismatic">
-    <parent link="base_link"/>
-    <child link="gripper_pole"/>
-    <limit effort="1000.0" lower="-${width*2-.02}" upper="0" velocity="0.5"/>
-    <origin rpy="0 0 0" xyz="${width-.01} 0 0.2"/>
-  </joint>
-  <link name="gripper_pole">
-    <visual>
-      <geometry>
-        <cylinder length="${polelen}" radius="0.01"/>
-      </geometry>
-      <origin xyz="${polelen/2} 0 0" rpy="0 ${pi/2} 0 "/>
-    </visual>
-    <collision>
-      <geometry>
-        <cylinder length="${polelen}" radius="0.01"/>
-      </geometry>
-      <origin xyz="${polelen/2} 0 0" rpy="0 ${pi/2} 0 "/>
-    </collision>
-    <xacro:default_inertial mass="0.05"/>
-  </link>
-  <xacro:macro name="gripper" params="prefix reflect">
-    <joint name="${prefix}_gripper_joint" type="revolute">
-      <axis xyz="0 0 ${reflect}"/>
-      <limit effort="1000.0" lower="0.0" upper="0.548" velocity="0.5"/>
-      <origin rpy="0 0 0" xyz="${polelen} ${reflect*0.01} 0"/>
-      <parent link="gripper_pole"/>
-      <child link="${prefix}_gripper"/>
+    <link name="Ferramenta">
+        <visual>
+            <geometry>
+                <box size="${MedidaPadrao} ${MedidaPadrao} ${AlturaFerramenta}"/>
+            </geometry>
+            <material name="blue"/>
+            <origin xyz="0 0 ${-AlturaFerramenta/2}" />
+        </visual>
+    </link>
+    <joint name="Antebraco_to_Ferramenta" type="revolute">
+        <parent link="Antebraco"/>
+        <child link="Ferramenta"/>
+        <axis xyz="0 0 1"/>
+        <limit effort="1000.0" lower="0.0" upper="0.548" velocity="0.5"/>
+        <origin xyz="0 0 ${AlturaFerramenta}" />
     </joint>
-    <link name="${prefix}_gripper">
-      <visual>
-        <origin rpy="${(reflect-1)/2*pi} 0 0" xyz="0 0 0"/>
-        <geometry>
-          <mesh filename="package://urdf_tutorial/meshes/l_finger.dae"/>
-        </geometry>
-      </visual>
-      <collision>
-        <geometry>
-          <mesh filename="package://urdf_tutorial/meshes/l_finger.dae"/>
-        </geometry>
-        <origin rpy="${(reflect-1)/2*pi} 0 0" xyz="0 0 0"/>
-      </collision>
-      <xacro:default_inertial mass="0.05"/>
-    </link>
-    <joint name="${prefix}_tip_joint" type="fixed">
-      <parent link="${prefix}_gripper"/>
-      <child link="${prefix}_tip"/>
-    </joint>
-    <link name="${prefix}_tip">
-      <visual>
-        <origin rpy="${(reflect-1)/2*pi} 0 0" xyz="0.09137 0.00495 0"/>
-        <geometry>
-          <mesh filename="package://urdf_tutorial/meshes/l_finger_tip.dae"/>
-        </geometry>
-      </visual>
-      <collision>
-        <geometry>
-          <mesh filename="package://urdf_tutorial/meshes/l_finger_tip.dae"/>
-        </geometry>
-        <origin rpy="${(reflect-1)/2*pi} 0 0" xyz="0.09137 0.00495 0"/>
-      </collision>
-      <xacro:default_inertial mass="0.05"/>
-    </link>
-  </xacro:macro>
-  <xacro:gripper prefix="left" reflect="1" />
-  <xacro:gripper prefix="right" reflect="-1" />
-  <link name="head">
-    <visual>
-      <geometry>
-        <sphere radius="${width}"/>
-      </geometry>
-      <material name="white"/>
-    </visual>
-    <collision>
-      <geometry>
-        <sphere radius="${width}"/>
-      </geometry>
-    </collision>
-    <xacro:default_inertial mass="2"/>
-  </link>
-  <joint name="head_swivel" type="continuous">
-    <parent link="base_link"/>
-    <child link="head"/>
-    <axis xyz="0 0 1"/>
-    <origin xyz="0 0 ${bodylen/2}"/>
-  </joint>
-  <link name="box">
-    <visual>
-      <geometry>
-        <box size="0.08 0.08 0.08"/>
-      </geometry>
-      <material name="blue"/>
-      <origin xyz="-0.04 0 0"/>
-    </visual>
-    <collision>
-      <geometry>
-        <box size="0.08 0.08 0.08"/>
-      </geometry>
-    </collision>
-    <xacro:default_inertial mass="1"/>
-  </link>
-  <joint name="tobox" type="fixed">
-    <parent link="head"/>
-    <child link="box"/>
-    <origin xyz="${.707*width+0.04} 0 ${.707*width}"/>
-  </joint>
 </robot>

Commit message: Parametros DH
Implementaçãos dos parametros de DH em arquivo URDF

File: urdf/bres.urdf.xacro (robot description, xacro)
@@ -1,10 +1,34 @@
 <?xml version="1.0"?>
 <robot name="macroed" xmlns:xacro="http://ros.org/wiki/xacro">
-    <xacro:property name="AlturaBase" value="0.0965" />
-    <xacro:property name="AlturaOmbro" value="0.0750" />
+    <!-- Parametros DH -->
+    <xacro:property name="Elo1_theta" value="livre" />
+    <xacro:property name="Elo1_alfa" value="${pi}" />
+    <xacro:property name="Elo1_a" value="0" />
+    <xacro:property name="Elo1_d" value="0.5" />
+    <xacro:property name="Elo2_theta" value="0" />
+    <xacro:property name="Elo2_alfa" value="0" />
+    <xacro:property name="Elo2_a" value="0.25" />
+    <xacro:property name="Elo2_d" value="livre" />
+    <xacro:property name="Elo3_theta" value="livre" />
+    <xacro:property name="Elo3_alfa" value="0" />
+    <xacro:property name="Elo3_a" value="0" />
+    <xacro:property name="Elo3_d" value="0.1" />
+    <xacro:property name="Elo4_theta" value="livre" />
+    <xacro:property name="Elo4_alfa" value="0" />
+    <xacro:property name="Elo4_a" value="0.25" />
+    <xacro:property name="Elo4_d" value="0.1" />
+    <!-- Medidas de colisao -->
+    <xacro:property name="RaioBase" value="0.1000" />
+    <xacro:property name="AlturaBase" value="0.1000" />
+    <xacro:property name="AlturaOmbro" value="0.3000" />
+    <xacro:property name="larguraOmbro" value="0.1100" />
+    <xacro:property name="ComprimentoOmbro" value="0.1500" />
+    <xacro:property name="RaioBraco" value="0.1000" />
     <xacro:property name="AlturaBraco" value="0.0850" />
-    <xacro:property name="AlturaAntebraco" value="0.0740" />
-    <xacro:property name="AlturaFerramenta" value="0.0300" />
-    <xacro:property name="MedidaPadrao" value="0.1000" />
+    <xacro:property name="RaioAntebraco" value="0.0800" />
+    <xacro:property name="AlturaAntebraco" value="0.0800" />
+    <xacro:property name="AlturaFerramenta" value="0.0500" />
+    <xacro:property name="larguraFerramenta" value="0.0500" />
+    <xacro:property name="ComprimentoFerramenta" value="0.0500" />
     <material name="blue">
     <color rgba="0 0 0.8 1"/>
@@ -13,51 +37,61 @@
         <visual>
             <geometry>
-                <cylinder radius="${MedidaPadrao}" length="${AlturaBase}"/>
+                <mesh filename="package://bres/meshes/3d_base.stl"/>
             </geometry>
             <material name="blue"/>
             <origin xyz="0 0 ${AlturaBase/2}" />
         </visual>
+        <collision>
+            <geometry>
+                <cylinder radius="${RaioBase}" length="${AlturaBase}"/>
+            </geometry>
+            <material name="blue"/>
+            <origin xyz="0 0 ${AlturaBase/2}" />
+        </collision>
     </link>
     <link name="Ombro">
         <visual>
             <geometry>
-                <box size="${MedidaPadrao} ${MedidaPadrao} ${AlturaOmbro}"/>
+                <box size="${ComprimentoOmbro} ${larguraOmbro} ${AlturaOmbro}"/>
             </geometry>
             <material name="blue"/>
-            <origin xyz="0 0 ${-AlturaOmbro/2}" />
+            <origin xyz="0 0 ${AlturaOmbro/2}" />
         </visual>
     </link>
-    <joint name="base_to_Ombro" type="prismatic">
+    <!-- Junta 1 -->
+    <joint name="base_to_Ombro" type="revolute">
         <parent link="base_link"/>
         <child link="Ombro"/>
-        <limit effort="1000.0" lower="-0.2500" upper="-0.1000" velocity="0.5"/>
         <axis xyz="0 0 1"/>
-        <origin xyz="0 0 ${AlturaBase}" rpy="${pi} 0 0" />
+        <limit effort="1000.0" lower="0.0" upper="0.548" velocity="0.5"/>
+        <origin xyz="${Elo1_a} 0 ${Elo1_d}" rpy="${Elo1_alfa} 0 0" />
     </joint>
     <link name="Braco">
         <visual>
             <geometry>
-                <cylinder radius="${MedidaPadrao}" length="${AlturaBraco}"/>
+                <cylinder radius="${RaioBraco}" length="${AlturaBraco}"/>
             </geometry>
             <material name="blue"/>
-            <origin xyz="0 0 ${-AlturaBraco/2}" />
+            <origin xyz="0 0 ${AlturaBraco/2}" />
         </visual>
     </link>
-    <joint name="Ombro_to_Braco" type="revolute">
+   <!-- Junta 2 -->
+    <joint name="Ombro_to_Braco" type="prismatic">
         <parent link="Ombro"/>
         <child link="Braco"/>
         <axis xyz="0 0 1"/>
-        <limit effort="1000.0" lower="0.0" upper="0.548" velocity="0.5"/>
-        <origin xyz="0.2500 0 0" />
+        <limit effort="1000.0" lower="0" upper="0.1" velocity="0.5"/>
+        <origin xyz="${Elo2_a} 0 0" rpy="${Elo2_alfa} 0 ${Elo2_theta}" />
     </joint>
     <link name="Antebraco">
         <visual>
             <geometry>
-                <cylinder radius="${MedidaPadrao}" length="${AlturaAntebraco}"/>
+                <cylinder radius="${RaioAntebraco}" length="${AlturaAntebraco}"/>
             </geometry>
             <material name="blue"/>
-            <origin xyz="0 0 ${-AlturaAntebraco/2}" />
+            <origin xyz="0 0 ${AlturaAntebraco/2}" />
         </visual>
     </link>
+    <!-- Junta 3 -->
     <joint name="Braco_to_Antebraco" type="revolute">
         <parent link="Braco"/>
@@ -65,15 +99,16 @@
         <axis xyz="0 0 1"/>
         <limit effort="1000.0" lower="0.0" upper="0.548" velocity="0.5"/>
-        <origin xyz="0.2500 0 0" />
+        <origin xyz="${Elo3_a} 0 ${Elo3_d}" rpy="${Elo3_alfa} 0 0" />
     </joint>
     <link name="Ferramenta">
         <visual>
             <geometry>
-                <box size="${MedidaPadrao} ${MedidaPadrao} ${AlturaFerramenta}"/>
+                <box size="${ComprimentoFerramenta} ${larguraFerramenta} ${AlturaFerramenta}"/>
             </geometry>
             <material name="blue"/>
-            <origin xyz="0 0 ${-AlturaFerramenta/2}" />
+            <origin xyz="0 0 ${AlturaFerramenta/2}" />
         </visual>
     </link>
+    <!-- Junta 4 -->
     <joint name="Antebraco_to_Ferramenta" type="revolute">
         <parent link="Antebraco"/>
@@ -81,5 +116,5 @@
         <axis xyz="0 0 1"/>
         <limit effort="1000.0" lower="0.0" upper="0.548" velocity="0.5"/>
-        <origin xyz="0 0 ${AlturaFerramenta}" />
+        <origin xyz="${Elo4_a} 0 ${Elo4_d}" rpy="${Elo4_alfa} 0 0" />
     </joint>
 </robot>

Commit message: CAD
Implementacao do cad com ajuste de constantes

File: urdf/bres.urdf.xacro (robot description, xacro)
@@ -5,5 +5,5 @@
     <xacro:property name="Elo1_alfa" value="${pi}" />
     <xacro:property name="Elo1_a" value="0" />
-    <xacro:property name="Elo1_d" value="0.5" />
+    <xacro:property name="Elo1_d" value="0.33" />
     <xacro:property name="Elo2_theta" value="0" />
     <xacro:property name="Elo2_alfa" value="0" />
@@ -16,10 +16,10 @@
     <xacro:property name="Elo4_theta" value="livre" />
     <xacro:property name="Elo4_alfa" value="0" />
-    <xacro:property name="Elo4_a" value="0.25" />
+    <xacro:property name="Elo4_a" value="0.13" />
     <xacro:property name="Elo4_d" value="0.1" />
     <!-- Medidas de colisao -->
     <xacro:property name="RaioBase" value="0.1000" />
     <xacro:property name="AlturaBase" value="0.1000" />
-    <xacro:property name="AlturaOmbro" value="0.3000" />
+    <xacro:property name="AlturaOmbro" value="0.2500" />
     <xacro:property name="larguraOmbro" value="0.1100" />
     <xacro:property name="ComprimentoOmbro" value="0.1500" />
@@ -31,4 +31,6 @@
     <xacro:property name="larguraFerramenta" value="0.0500" />
     <xacro:property name="ComprimentoFerramenta" value="0.0500" />
+    <!-- Escala para arquivos .STL -->
+    <xacro:property name="EscalaSTL" value="0.001 0.001 0.001" />
     <material name="blue">
     <color rgba="0 0 0.8 1"/>
@@ -37,8 +39,8 @@
         <visual>
             <geometry>
-                <mesh filename="package://bres/meshes/3d_base.stl"/>
+                <mesh filename="package://bres/meshes/Base.stl" scale="${EscalaSTL}" />
             </geometry>
             <material name="blue"/>
-            <origin xyz="0 0 ${AlturaBase/2}" />
+            <origin xyz="0 0 ${AlturaBase/2}" rpy="0 0 ${pi/2}" />
         </visual>
         <collision>
@@ -53,9 +55,16 @@
         <visual>
             <geometry>
+                <mesh filename="package://bres/meshes/Eixo_Z.stl" scale="${EscalaSTL}" />
+            </geometry>
+            <material name="blue"/>
+            <origin xyz="0 0 ${AlturaOmbro}" rpy="${pi} 0 ${pi/2}" />
+        </visual>
+        <collision>
+            <geometry>
                 <box size="${ComprimentoOmbro} ${larguraOmbro} ${AlturaOmbro}"/>
             </geometry>
             <material name="blue"/>
             <origin xyz="0 0 ${AlturaOmbro/2}" />
-        </visual>
+        </collision>
     </link>
     <!-- Junta 1 -->
@@ -70,9 +79,16 @@
         <visual>
             <geometry>
+                <mesh filename="package://bres/meshes/Braco.stl" scale="${EscalaSTL}" />
+            </geometry>
+            <material name="blue"/>
+            <origin xyz="${0.05-Elo2_a} 0 ${AlturaBraco}" rpy="${pi} 0 ${-pi/2}" />
+        </visual>
+        <collision>
+            <geometry>
                 <cylinder radius="${RaioBraco}" length="${AlturaBraco}"/>
             </geometry>
             <material name="blue"/>
             <origin xyz="0 0 ${AlturaBraco/2}" />
-        </visual>
+        </collision>
     </link>
    <!-- Junta 2 -->
@@ -87,9 +103,16 @@
         <visual>
             <geometry>
+                <mesh filename="package://bres/meshes/Antebraco.stl" scale="${EscalaSTL}" />
+            </geometry>
+            <material name="blue"/>
+            <origin xyz="${Elo3_a} 0 0" rpy="${pi} 0 ${-pi/2}" />
+        </visual>
+        <collision>
+            <geometry>
                 <cylinder radius="${RaioAntebraco}" length="${AlturaAntebraco}"/>
             </geometry>
             <material name="blue"/>
             <origin xyz="0 0 ${AlturaAntebraco/2}" />
-        </visual>
+        </collision>
     </link>
     <!-- Junta 3 -->
@@ -107,6 +130,13 @@
             </geometry>
             <material name="blue"/>
+            <origin xyz="0 0 ${-AlturaFerramenta/2}" />
+        </visual>
+        <collision>
+            <geometry>
+                <box size="${ComprimentoFerramenta} ${larguraFerramenta} ${AlturaFerramenta}"/>
+            </geometry>
+            <material name="blue"/>
             <origin xyz="0 0 ${AlturaFerramenta/2}" />
-        </visual>
+        </collision>
     </link>
     <!-- Junta 4 -->
